File: headphone_amp.kicad_pcb (KiCad board)
At the start: 2 copper layers, 81 parts, among them J1 btn, J10 Conn_01x04, J2 AUX_IN, J3 IN, J4 pangea_cp16, J5 USB_A, J6 OUT, J7 PWR, U1 NE5532, U3 NE5532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

Commit message: working version
Parts:
- removed R3: 100k, Resistor_SMD:R_1206_3216Metric
- removed R4: 0, Resistor_SMD:R_1206_3216Metric
- removed R6: 0, Resistor_SMD:R_2512_6332Metric
- removed RV1: 10K, Connector_PinSocket_2.54mm:PinSocket_1x03_P2.54mm_Vertical
- moved R36 45.7 mm to (86.0, 71.0), turned to 180 degrees
- moved R7 29.8 mm to (59.5, 50.0), turned to 270 degrees
- moved C6 23.2 mm to (60.5, 45.0), turned to 270 degrees
- moved R10 17.5 mm to (62.0, 40.5), turned to 270 degrees
- moved C1 11.7 mm to (79.0, 77.0), turned to 270 degrees
- moved C2 11.0 mm to (75.5, 76.0), turned to 270 degrees
- moved J10 10.4 mm to (52.5, 90.5), turned to 90 degrees
- moved R37 10.3 mm to (70.5, 63.5), turned to 90 degrees
- moved D1 7.28 mm to (70.0, 67.5)
- moved C5 2.55 mm to (80.5, 63.0)
- moved R23 2.50 mm to (83.5, 64.0)
- moved C3 2.06 mm to (87.0, 63.0)
- moved C13 2.06 mm to (57.5, 45.0)
- moved R1 1.50 mm to (77.0, 64.0), turned to 90 degrees
Connections:
- J3 pad 1: Net-(J3-Pad1) -> Net-(C6-Pad2)
Routing:
- net Net-(R3-Pad2): track 38.1 -> 0.00 mm
- net /ps4: track 24.3 -> 5.51 mm
- net Net-(J3-Pad1): track 15.4 -> 0.00 mm
- net /ps3: track 20.7 -> 5.51 mm
- net Net-(C12-Pad2): track 34.5 -> 19.7 mm
- net /ps2: track 17.1 -> 5.51 mm
- net /ps1: track 13.5 -> 5.51 mm
- net +4V: track 157.8 -> 152.8 mm
- net GND: track 31.6 -> 26.7 mm, vias 6 -> 8
- net Net-(C12-Pad1): track 73.5 -> 76.9 mm
- net +9V: track 183.0 -> 181.1 mm
- net /aux_r: track 77.9 -> 76.1 mm
- net Net-(C6-Pad2): track 6.95 -> 8.74 mm
- net Net-(R23-Pad2): track 4.69 -> 3.65 mm
- net Net-(C3-Pad1): track 3.83 -> 4.50 mm
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Other:
- net class power: clearance 0.6 -> 0.5; trace_width 0.8 -> 0.6
