File: headphone_amp.sch (KiCad schematic (older format))
At the start: 81 parts, among them J1 btn, J10 Conn_01x04, J2 AUX_IN, J3 IN, J4 pangea_cp16, J5 USB_A, J6 OUT, J7 PWR, U1 NE5532, U3 NE5532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

Commit message: working version
Parts:
- removed R3: 100k, Resistor_SMD:R_1206_3216Metric, symbol Device:R
- removed R4: 0, Resistor_SMD:R_1206_3216Metric, symbol Device:R
- removed R6: 0, Resistor_SMD:R_2512_6332Metric, symbol Device:R
- removed RV1: 10K, Connector_PinSocket_2.54mm:PinSocket_1x03_P2.54mm_Vertical, symbol Device:POT
- added U?: NE5532, symbol Amplifier_Operational:NE5532
- RV2: symbol Device:POT_Dual -> Device:R_POT_Dual
Connections:
- wire segments 218 -> 208
Other:
- moved on the sheet: J3
Changed lines of the file:
@@
 L Connector_Specialized:Audio-Jack-3_3Switches J3
 U 1 1 5AD505BE
-P 1150 5550
-F 0 "J3" H 1154 5975 50  0000 C CNN
-F 1 "IN" H 1154 5884 50  0000 C CNN
-F 2 "footprint:Jack6P" H 1400 5650 50  0001 C CNN
-F 3 "~" H 1400 5650 50  0001 C CNN
-	1    1150 5550
+P 2000 5950
+F 0 "J3" H 2004 6375 50  0000 C CNN
+F 1 "IN" H 2004 6284 50  0000 C CNN
+F 2 "footprint:Jack6P" H 2250 6050 50  0001 C CNN
+F 3 "~" H 2250 6050 50  0001 C CNN
+	1    2000 5950
 	1    0    0    -1
 $EndComp
@@
 L power:GND #PWR09
 U 1 1 5AD508BF
-P 1700 5400
-F 0 "#PWR09" H 1700 5150 50  0001 C CNN
-F 1 "GND" H 1705 5227 50  0000 C CNN
-F 2 "" H 1700 5400 50  0001 C CNN
-F 3 "" H 1700 5400 50  0001 C CNN
-	1    1700 5400
-	1    0    0    -1
-$EndComp
-NoConn ~ 1350 5650
-$Comp
-L Device:R R3
-U 1 1 5AD61D5C
-P 2250 6100
-F 0 "R3" H 2150 6050 50  0000 C CNN
-F 1 "100k" H 2400 6050 50  0000 C CNN
-F 2 "Resistor_SMD:R_1206_3216Metric" V 2180 6100 50  0001 C CNN
-F 3 "" H 2250 6100 50  0001 C CNN
-	1    2250 6100
-	1    0    0    -1
-$EndComp
-$Comp
-L Device:POT RV1
-U 1 1 5AD65199
-P 2250 6400
-F 0 "RV1" H 2180 6446 50  0000 R CNN
-F 1 "10K" H 2180 6355 50  0000 R CNN
-F 2 "Connector_PinSocket_2.54mm:PinSocket_1x03_P2.54mm_Vertical" H 2250 6400 50  0001 C CNN
-F 3 "" H 2250 6400 50  0001 C CNN
-	1    2250 6400
-	1    0    0    -1
-$EndComp
-$Comp
-L power:GND #PWR014
-U 1 1 5AD6548D
-P 2250 6550
-F 0 "#PWR014" H 2250 6300 50  0001 C CNN
-F 1 "GND" H 2255 6377 50  0000 C CNN
-F 2 "" H 2250 6550 50  0001 C CNN
-F 3 "" H 2250 6550 50  0001 C CNN
-	1    2250 6550
-	1    0    0    -1
-$EndComp
+P 2550 5800
+F 0 "#PWR09" H 2550 5550 50  0001 C CNN
+F 1 "GND" H 2555 5627 50  0000 C CNN
+F 2 "" H 2550 5800 50  0001 C CNN
+F 3 "" H 2550 5800 50  0001 C CNN
+	1    2550 5800
+	1    0    0    -1
+$EndComp
+NoConn ~ 2200 6050
 $Comp
 L Device:R R7
@@
 $EndComp
 Wire Wire Line
-	2400 6400 2550 6400
-Wire Wire Line
-	2550 6400 2550 6150
-Wire Wire Line
 	2850 6300 2850 6150
-Wire Wire Line
-	2550 6150 2850 6150
 Connection ~ 2850 6150
 Wire Wire Line
@@
 ain
 $Comp
-L Device:POT_Dual RV2
+L Device:R_POT_Dual RV2
 U 1 1 5ADF2BC5
 P 7650 2400
@@
 	8900 2800 9150 2800
 $Comp
-L Device:R R4
-U 1 1 5AD9B1D0
-P 9600 2650
-F 0 "R4" V 9700 2650 50  0000 C CNN
-F 1 "0" V 9500 2650 50  0000 C CNN
-F 2 "Resistor_SMD:R_1206_3216Metric" V 9530 2650 50  0001 C CNN
-F 3 "" H 9600 2650 50  0001 C CNN
-	1    9600 2650
-	-1   0    0    1
-$EndComp
-$Comp
-L power:+4V #PWR0108
-U 1 1 5AD9B322
-P 9600 2500
-F 0 "#PWR0108" H 9600 2350 50  0001 C CNN
-F 1 "+4V" H 9615 2673 50  0000 C CNN
-F 2 "" H 9600 2500 50  0001 C CNN
-F 3 "" H 9600 2500 50  0001 C CNN
-	1    9600 2500
-	1    0    0    -1
-$EndComp
-$Comp
-L power:+4V #PWR0109
-U 1 1 5AD9B461
-P 9850 2600
-F 0 "#PWR0109" H 9850 2450 50  0001 C CNN
-F 1 "+4V" H 9865 2773 50  0000 C CNN
-F 2 "" H 9850 2600 50  0001 C CNN
-F 3 "" H 9850 2600 50  0001 C CNN
-	1    9850 2600
-	1    0    0    -1
-$EndComp
-Wire Wire Line
-	9600 2800 9600 2850
-Wire Wire Line
-	9600 2850 9850 2850
-Wire Wire Line
-	9850 2850 9850 2600
-$Comp
-L power:+4V #PWR0110
-U 1 1 5ADA4F2B
-P 10100 2500
-F 0 "#PWR0110" H 10100 2350 50  0001 C CNN
-F 1 "+4V" H 10115 2673 50  0000 C CNN
-F 2 "" H 10100 2500 50  0001 C CNN
-F 3 "" H 10100 2500 50  0001 C CNN
-	1    10100 2500
-	1    0    0    -1
-$EndComp
-$Comp
-L power:+4V #PWR0111
-U 1 1 5ADA4F31
-P 10350 2600
-F 0 "#PWR0111" H 10350 2450 50  0001 C CNN
-F 1 "+4V" H 10365 2773 50  0000 C CNN
-F 2 "" H 10350 2600 50  0001 C CNN
-F 3 "" H 10350 2600 50  0001 C CNN
-	1    10350 2600
-	1    0    0    -1
-$EndComp
-Wire Wire Line
-	10100 2800 10100 2850
-Wire Wire Line
-	10100 2850 10350 2850
-Wire Wire Line
-	10350 2850 10350 2600
-$Comp
 L Device:R R30
 U 1 1 5ADAF397
@@
 Wire Wire Line
 	2250 4950 2150 4950
-Connection ~ 2150 4950
 Wire Wire Line
 	1850 4350 1800 4350
@@
 Wire Wire Line
 	6300 2400 6300 2200
-Connection ~ 5950 2400
-Wire Wire Line
-	1350 5350 1700 5350
-Wire Wire Line
-	1700 5350 1700 5400
-NoConn ~ 1350 5550
+Wire Wire Line
+	2200 5750 2550 5750
+Wire Wire Line
+	2550 5750 2550 5800
+NoConn ~ 2200 5950
 $Comp
 L power:GND #PWR0119
 U 1 1 5ADDC4E0
-P 1550 6000
-F 0 "#PWR0119" H 1550 5750 50  0001 C CNN
-F 1 "GND" H 1555 5827 50  0000 C CNN
-F 2 "" H 1550 6000 50  0001 C CNN
-F 3 "" H 1550 6000 50  0001 C CNN
-	1    1550 6000
-	1    0    0    -1
-$EndComp
-Wire Wire Line
-	1350 5850 1550 5850
-Wire Wire Line
-	1550 5850 1550 6000
-Wire Wire Line
-	2250 5750 2250 5950
+P 2400 6400
+F 0 "#PWR0119" H 2400 6150 50  0001 C CNN
+F 1 "GND" H 2405 6227 50  0000 C CNN
+F 2 "" H 2400 6400 50  0001 C CNN
+F 3 "" H 2400 6400 50  0001 C CNN
+	1    2400 6400
+	1    0    0    -1
+$EndComp
+Wire Wire Line
+	2200 6250 2400 6250
+Wire Wire Line
+	2400 6250 2400 6400
 $Comp
 L power:+9V #PWR0120
@@
 	6900 2400 7100 2400
 Wire Wire Line
-	1350 5750 2250 5750
-Wire Wire Line
 	4800 6700 5250 6700
-$Comp
-L Device:R R6
-U 1 1 5AE6CFF7
-P 10100 2650
-F 0 "R6" V 10200 2650 50  0000 C CNN
-F 1 "0" V 10000 2650 50  0000 C CNN
-F 2 "Resistor_SMD:R_2512_6332Metric" V 10030 2650 50  0001 C CNN
-F 3 "" H 10100 2650 50  0001 C CNN
-	1    10100 2650
-	-1   0    0    1
-$EndComp
-NoConn ~ 1350 5450
+NoConn ~ 2200 5850
+Wire Wire Line
+	2200 6150 2850 6150
+$Comp
+L Amplifier_Operational:NE5532 U?
+U 3 1 5B0F7DE1
+P 8600 4800
+F 0 "U?" H 8558 4846 50  0000 L CNN
+F 1 "NE5532" H 8558 4755 50  0000 L CNN
+F 2 "" H 8600 4800 50  0001 C CNN
+F 3 "http://www.ti.com/lit/ds/symlink/ne5532.pdf" H 8600 4800 50  0001 C CNN
+	3    8600 4800
+	1    0    0    -1
+$EndComp
 $EndSCHEMATC
